File: SmartTherm-PCB.kicad_sch (KiCad schematic)
At the start: 22 parts, among them J1 Junkers, J2 Display - Sensor, J3 Ext LDR, Q1 BC546, U1 WeMos D1 mini, U2 ILD74, U3 LM358

Commit message: update BOM
Parts:
- C1: manufacturerPartNumber (none) -> RCEC72A475MWM1H03A; mouserPartNumber (none) -> 81-RCEC72A475MWM1H3A
- C2: manufacturerPartNumber (none) -> FA22X7R2J104KNU06; mouserPartNumber (none) -> 810-FA22X7R2J104KNU6
- H1, H2, H3, H4: manufacturerPartNumber (none) -> na; mouserPartNumber (none) -> na
- J1: manufacturerPartNumber (none) -> 1711042; mouserPartNumber (none) -> 651-1711042
- J2: manufacturerPartNumber (none) -> 1730052; mouserPartNumber (none) -> 651-1730052
- J3: manufacturerPartNumber (none) -> 1711026; mouserPartNumber (none) -> 651-1711026
- Q1: manufacturerPartNumber (none) -> BC546A; mouserPartNumber (none) -> 637-BC546A
- R10: manufacturerPartNumber (none) -> CCF554K70FKE36; mouserPartNumber (none) -> 71-CCF554K70FKE36
- R8, R9: manufacturerPartNumber (none) -> CCF551K00FKE36; mouserPartNumber (none) -> 71-CCF551K00FKE36
- U2: manufacturerPartNumber (none) -> ILD74; mouserPartNumber (none) -> 782-ILD74
- U3: manufacturerPartNumber (none) -> LM358N/NOPB; mouserPartNumber (none) -> 926-LM358N/NOPB

Commit message: updates to pass ERC/DRC
Parts:
- R1: footprint Resistor_THT:R_Axial_DIN0207_L6.3mm_D2.5mm_P10.16mm_Horizontal -> 1projectLibrary:R_Axial_DIN0207_L6.3mm_D2.5mm_P10.16mm_Horizontal; manufacturerPartNumber (none) -> RL07S332GB14; mouserPartNumber (none) -> 71-RL07S-G-3.3K
- R10: footprint Resistor_THT:R_Axial_DIN0207_L6.3mm_D2.5mm_P10.16mm_Horizontal -> 1projectLibrary:R_Axial_DIN0207_L6.3mm_D2.5mm_P10.16mm_Horizontal; manufacturerPartNumber CCF554K70FKE36 -> RL07S472GB14; mouserPartNumber 71-CCF554K70FKE36 -> 71-RL07S-G-4.7K
- R3, R4: footprint Resistor_THT:R_Axial_DIN0207_L6.3mm_D2.5mm_P10.16mm_Horizontal -> 1projectLibrary:R_Axial_DIN0207_L6.3mm_D2.5mm_P10.16mm_Horizontal; manufacturerPartNumber (none) -> RL07S103GB14; mouserPartNumber (none) -> 71-RL07S-G-10K
- R5: footprint Resistor_THT:R_Axial_DIN0207_L6.3mm_D2.5mm_P10.16mm_Horizontal -> 1projectLibrary:R_Axial_DIN0207_L6.3mm_D2.5mm_P10.16mm_Horizontal; manufacturerPartNumber (none) -> RL07S223GB14; mouserPartNumber (none) -> 71-RL07S-G-22K
- R6: footprint Resistor_THT:R_Axial_DIN0207_L6.3mm_D2.5mm_P10.16mm_Horizontal -> 1projectLibrary:R_Axial_DIN0207_L6.3mm_D2.5mm_P10.16mm_Horizontal; manufacturerPartNumber (none) -> RL07S473GB14; mouserPartNumber (none) -> 71-RL07S-G-47K
- R7: footprint Resistor_THT:R_Axial_DIN0207_L6.3mm_D2.5mm_P10.16mm_Horizontal -> 1projectLibrary:R_Axial_DIN0207_L6.3mm_D2.5mm_P10.16mm_Horizontal; manufacturerPartNumber (none) -> RL07S471GB14; mouserPartNumber (none) -> 71-RL07S-G-470
- R8, R9: footprint Resistor_THT:R_Axial_DIN0207_L6.3mm_D2.5mm_P10.16mm_Horizontal -> 1projectLibrary:R_Axial_DIN0207_L6.3mm_D2.5mm_P10.16mm_Horizontal; manufacturerPartNumber CCF551K00FKE36 -> RL07S102GB14; mouserPartNumber 71-CCF551K00FKE36 -> 71-RL07S-G-1K
- U1: footprint Module:WEMOS_D1_mini_light -> 1projectLibrary:WEMOS_D1_mini_light
Connections:
- net 24Present renamed 24V-Present
Other:
- moved on the sheet: R1, U2A

Commit message: footprint updates
Parts:
- C1, C2: footprint Capacitor_THT:C_Disc_D4.7mm_W2.5mm_P5.00mm -> 1projectLibrary:C_Disc_D4.7mm_W2.5mm_P5.00mm
- J1: footprint TerminalBlock_Phoenix:TerminalBlock_Phoenix_PT-1,5-4-5.0-H_1x04_P5.00mm_Horizontal -> 1projectLibrary:TerminalBlock_Junkers
- J3: footprint TerminalBlock_Phoenix:TerminalBlock_Phoenix_PT-1,5-2-5.0-H_1x02_P5.00mm_Horizontal -> 1projectLibrary:TerminalBlock_LDR
- Q1: footprint Package_TO_SOT_THT:TO-92L_Inline_Wide -> 1projectLibrary:TO-92L_Inline_Wide
- U2, U3: footprint Package_DIP:DIP-8_W7.62mm -> 1projectLibrary:DIP-8_W7.62mm
Changed lines of the file:
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@@
 			)
 		)
-		(property "Footprint" "Package_DIP:DIP-8_W7.62mm"
+		(property "Footprint" "1projectLibrary:DIP-8_W7.62mm"
 			(at 146.05 97.79 0)
 			(effects
@@
 			)
 		)
-		(property "Footprint" "Package_DIP:DIP-8_W7.62mm"
+		(property "Footprint" "1projectLibrary:DIP-8_W7.62mm"
 			(at 135.89 110.49 0)
 			(effects
@@
 			)
 		)
-		(property "Footprint" "Package_DIP:DIP-8_W7.62mm"
+		(property "Footprint" "1projectLibrary:DIP-8_W7.62mm"
 			(at 193.04 93.98 0)
 			(effects
@@
 			)
 		)
-		(property "Footprint" "Package_DIP:DIP-8_W7.62mm"
+		(property "Footprint" "1projectLibrary:DIP-8_W7.62mm"
 			(at 224.79 96.52 0)
 			(effects
@@
 			)
 		)
-		(property "Footprint" "Package_DIP:DIP-8_W7.62mm"
+		(property "Footprint" "1projectLibrary:DIP-8_W7.62mm"
 			(at 255.27 96.52 0)
 			(effects
@@
 			)
 		)
-		(property "Footprint" "Package_TO_SOT_THT:TO-92L_Inline_Wide"
+		(property "Footprint" "1projectLibrary:TO-92L_Inline_Wide"
 			(at 179.07 104.775 0)
 			(effects
@@
 			)
 		)
-		(property "Footprint" "Capacitor_THT:C_Disc_D4.7mm_W2.5mm_P5.00mm"
+		(property "Footprint" "1projectLibrary:C_Disc_D4.7mm_W2.5mm_P5.00mm"
 			(at 241.6048 120.65 0)
 			(effects
@@
 			)
 		)
-		(property "Footprint" "Capacitor_THT:C_Disc_D4.7mm_W2.5mm_P5.00mm"
+		(property "Footprint" "1projectLibrary:C_Disc_D4.7mm_W2.5mm_P5.00mm"
 			(at 211.1248 120.65 0)
 			(effects
@@
 			)
 		)
-		(property "Footprint" "TerminalBlock_Phoenix:TerminalBlock_Phoenix_PT-1,5-4-5.0-H_1x04_P5.00mm_Horizontal"
+		(property "Footprint" "1projectLibrary:TerminalBlock_Junkers"
 			(at 269.24 69.85 0)
 			(effects
@@
 			)
 		)
-		(property "Footprint" "TerminalBlock_Phoenix:TerminalBlock_Phoenix_PT-1,5-2-5.0-H_1x02_P5.00mm_Horizontal"
+		(property "Footprint" "1projectLibrary:TerminalBlock_LDR"
 			(at 107.95 72.39 0)
 			(effects
